File: boards/board1/kicad/access.kicad_sch (KiCad schematic)
At the start: 29 parts, among them J12 1989803 / bus terminals, J13 GW GND, J14 SAM0 GND, J15 SAM1 GND, J16 SAM2 GND, J17 POWER GND, J18 BUS GND

Commit message: High-level layout done
Parts:
- removed TP13: UART_MD, TestPoint:TestPoint_Pad_D2.0mm, symbol Connector:TestPoint
- removed TP14: RS485_A, TestPoint:TestPoint_Pad_D2.0mm, symbol Connector:TestPoint
- removed TP15: RS485_B, TestPoint:TestPoint_Pad_D2.0mm, symbol Connector:TestPoint
- removed TP16: FD_CAN_A_H, TestPoint:TestPoint_Pad_D2.0mm, symbol Connector:TestPoint
- removed TP17: FD_CAN_A_L, TestPoint:TestPoint_Pad_D2.0mm, symbol Connector:TestPoint
- removed TP18: FD_CAN_B_H, TestPoint:TestPoint_Pad_D2.0mm, symbol Connector:TestPoint
- removed TP19: FD_CAN_B_L, TestPoint:TestPoint_Pad_D2.0mm, symbol Connector:TestPoint
- added J19: CAN A, Connector_PinHeader_2.54mm:PinHeader_1x02_P2.54mm_Vertical, symbol Connector_Generic:Conn_01x02
- added J20: CAN B, Connector_PinHeader_2.54mm:PinHeader_1x02_P2.54mm_Vertical, symbol Connector_Generic:Conn_01x02
- added J21: RS485, Connector_PinHeader_2.54mm:PinHeader_1x02_P2.54mm_Vertical, symbol Connector_Generic:Conn_01x02
- added J22: RING01, Connector_PinHeader_2.54mm:PinHeader_1x02_P2.54mm_Vertical, symbol Connector_Generic:Conn_01x02
- added J23: RING12, Connector_PinHeader_2.54mm:PinHeader_1x02_P2.54mm_Vertical, symbol Connector_Generic:Conn_01x02
- added J24: RING20, Connector_PinHeader_2.54mm:PinHeader_1x02_P2.54mm_Vertical, symbol Connector_Generic:Conn_01x02
- added J25: UART_MD, Connector_PinHeader_2.54mm:PinHeader_1x02_P2.54mm_Vertical, symbol Connector_Generic:Conn_01x02
Connections:
- net FD_CAN_A_H: now also J19.1 (Pin_1)
- net FD_CAN_A_L: now also J19.2 (Pin_2)
- net FD_CAN_B_H: now also J20.1 (Pin_1)
- net FD_CAN_B_L: now also J20.2 (Pin_2)
- net GND: now also J22.2 (Pin_2), J23.2 (Pin_2), J24.2 (Pin_2), J25.2 (Pin_2)
- net RS485_A: now also J21.1 (Pin_1)
- net RS485_B: now also J21.2 (Pin_2)
- net UART_MD: now also J25.1 (Pin_1)
- new net RING_01: J22.1 (Pin_1)
- new net RING_12: J23.1 (Pin_1)
- new net RING_20: J24.1 (Pin_1)
Other:
- note added: "PCB TEST PADS — power / reset / core rails (TP1–TP12)"
- note removed: "PCB TEST PADS (NO PURCHASED PART)"
- moved on the sheet: TP1, TP10, TP11, TP12, TP2, TP3, TP4, TP5, TP6, TP7, TP8, TP9
