File: boards/board1/kicad/board1.kicad_sch (KiCad schematic)
At the start: 22 parts, among them J1 USB-B1HSB6, U1 TPS22810DBVT, U2 TPS560430X3FDBVR, U3 MC74HC1G14DBVT1G

Commit message: First draft finished
Parts:
- removed C1: 1u / 25V, Capacitor_SMD:C_0805_2012Metric, symbol Device:C
- removed C10, C5, C8, C9: 100n, Capacitor_SMD:C_0805_2012Metric, symbol Device:C
- removed C2: 4u7 / 50V, Capacitor_SMD:C_0805_2012Metric, symbol Device:C
- removed C3: 47n, Capacitor_SMD:C_0805_2012Metric, symbol Device:C
- removed C4: 4u7, Capacitor_SMD:C_0805_2012Metric, symbol Device:C
- removed C6: 10u / 35V, Capacitor_SMD:C_1206_3216Metric, symbol Device:C
- removed C7: 22u / 16V, Capacitor_SMD:C_1210_3225Metric, symbol Device:C
- removed D1: SMF6.0A, Diode_SMD:D_SOD-123F, symbol Device:D
- removed D2: RCLAMP0504S.TCT, Package_TO_SOT_SMD:SOT-23-6, symbol RCLAMP0504S.TCT:RCLAMP0504S.TCT
- removed D3: Orange, LED_SMD:LED_0603_1608Metric, symbol Device:LED
- removed J1: USB-B1HSB6, Connector_USB:USB_B_OST_USB-B1HSxx_Horizontal, symbol Connector:USB_B
- removed L1: 12uH, Inductor_SMD:L_Bourns_SRN6045TA, symbol Device:L
- removed R1: 1R / pulse, Resistor_SMD:R_1206_3216Metric, symbol Device:R
- removed R2: 10k, Resistor_SMD:R_0805_2012Metric, symbol Device:R
- removed R3: 47k, Resistor_SMD:R_0805_2012Metric, symbol Device:R
- removed R4: 3k3, Resistor_SMD:R_0805_2012Metric, symbol Device:R
- removed U1: TPS22810DBVT, Package_TO_SOT_SMD:SOT-23-6, symbol TPS22810DBVT:TPS22810DBVT
- removed U2: TPS560430X3FDBVR, Package_TO_SOT_SMD:SOT-23-6, symbol TPS560430X3FDBVR:TPS560430X3FDBVR
- removed U3: MC74HC1G14DBVT1G, Package_TO_SOT_SMD:SOT-23-5, symbol MC74HC1G14DBVT1G:MC74HC1G14DBVT1G
Connections:
- no-connect marks 4 -> 0
Other:
- added sheet CAN A (can_a.kicad_sch)
- added sheet CAN B (can_b.kicad_sch)
- added sheet Gateway STM32G474 (gateway.kicad_sch)
- added sheet SAM0 (sam0.kicad_sch)
- added sheet SAM1 (sam1.kicad_sch)
- added sheet SAM2 (sam2.kicad_sch)
- added sheet Test access (access.kicad_sch)
- added sheet UART and external terminals (interfaces.kicad_sch)
- added sheet USB input and power (power.kicad_sch)
- note added: "02 USB input and power"
- note added: "03 USB bridge and VCP"
- note added: "04 Gateway STM32G474"
- note added: "05 SAM0"
- note added: "06 SAM1"
- note added: "07 SAM2"
- note added: "08 CAN A"
- note added: "09 CAN B"
- note added: "10 UART and external terminals"
- note added: "11 Test access"
- note added: "CAN A/B: GW + SAM0 + SAM1 + SAM2, eight PHYs. UART_MD: four receivers; one LV125 channel per transmitter. SAM ring: SAM0 -> SAM1 -> SAM2 -> SAM0. Each MCU: SWD, private debug UART, SYNC/TRIG and EVENT0/1."
- note added: "Four MCU bench prototype: two shared CAN-FD buses, multidrop UART and SAM ring. Active PC USB power, 500 mA configured budget. Independent FTDI controls the main 3.3 V rail."
- note added: "Named global nets join sheets; local analog nets stay within their sheet. Review PDF and checks describe draft-capture evidence. ERC, layout/DRC and hardware bring-up are separate stages. No PCB layout yet."
- note added: "WIRESPACES / BOARD 1 REV A"
- note removed: "3.3 V MAIN BUCK"
- note removed: "C4/C5: place at FTDI VREGIN (U4 pin 40)."
- note removed: "Fixed X3F: FB senses output directly. Keep CB-SW loop short; quiet FB route. No divider, catch diode or external compensation."
- note removed: "POWER INDICATOR"
- note removed: "PWREN_N low: main rail ON, VCP buffers enabled. High / floating: main rail OFF (ADR-040)."
- note removed: "Pin 5 VREF unconnected: internal TVS mode. Unused channels 4/6 unconnected. Place at J1. Route USB differential pair directly; avoid stubs."
- note removed: "USB CONFIGURATION / SUSPEND CONTROL"
- note removed: "USB DATA ESD"
- note removed: "USB shield bonds directly to GND at entry."
- note removed: "USB-B INPUT AND ATTACHMENT RAMP"
- note removed: "USB-only, active-PC bench operation. 500 mA configured input budget. Power/USB capture ends at GW_VCP_TX/RX/RTS_N/CTS_N. MCU, CAN, RS-485 and timing-header sections are not captured. No external reset supervisor or CBUS recovery circuitry."
- note removed: "USB_5V / USB_DM / USB_DP FTDI_3V3 / PWREN_N / 3V3_SYS Cross-sheet connections use named global nets."
- title: Board 1 - USB input and main power -> Board 1 - Rev A system overview

Commit message: High-level layout done
Other:
- sheet Gateway STM32G474 renamed Gateway STM32G473
- note added: "04 Gateway STM32G473"
- note added: "Named global nets join sheets; local analog nets stay within their sheet. Review PDF and checks describe draft-capture evidence. ERC, layout/DRC and hardware bring-up are separate stages. Initial PCB placement is unrouted."
- note removed: "04 Gateway STM32G474"
- note removed: "Named global nets join sheets; local analog nets stay within their sheet. Review PDF and checks describe draft-capture evidence. ERC, layout/DRC and hardware bring-up are separate stages. No PCB layout yet."
Changed lines of the file:
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@@
 (kicad_sch (version 20230121) (generator ws_hardware_capture) (paper "A3")
-(title_block (title "Board 1 - Rev A system overview") (date "2026-09-07") (rev "A-draft") (company "WireSpaces") (comment 1 "Rev A complete schematic draft - no PCB layout"))
+(title_block (title "Board 1 - Rev A system overview") (date "2026-09-07") (rev "A-draft") (company "WireSpaces") (comment 1 "Rev A schematic draft - PCB placement unrouted"))
 (text "WIRESPACES  /  BOARD 1 REV A" (at 22 22 0) (effects (font (size 2.5 2.5)) (justify left top)))
 (text "Four MCU bench prototype: two shared CAN-FD buses, multidrop UART and SAM ring.\nActive PC USB power, 500 mA configured budget. Independent FTDI controls the main 3.3 V rail." (at 22 36 0) (effects (font (size 1.5 1.5)) (justify left top)))
@@
 (sheet (at 153 63) (size 112 27) (stroke (width 0) (type solid)) (fill (color 0 0 0 0)) (property "Sheetname" "USB bridge and VCP" (at 153 62 0) (effects (font (size 1.27 1.27)) (justify left bottom))) (property "Sheetfile" "usb_bridge.kicad_sch" (at 153 91 0) (effects (font (size 1.0 1.0)) (justify left top))) (instances (project "board1" (path "/ab028fb1-c655-584d-9b32-a6ba9517f8a2" (page "3")))))
 (text "03  USB bridge and VCP" (at 158 72 0) (effects (font (size 1.4 1.4)) (justify left top)))
-(sheet (at 281 63) (size 112 27) (stroke (width 0) (type solid)) (fill (color 0 0 0 0)) (property "Sheetname" "Gateway STM32G474" (at 281 62 0) (effects (font (size 1.27 1.27)) (justify left bottom))) (property "Sheetfile" "gateway.kicad_sch" (at 281 91 0) (effects (font (size 1.0 1.0)) (justify left top))) (instances (project "board1" (path "/ab028fb1-c655-584d-9b32-a6ba9517f8a2" (page "4")))))
-(text "04  Gateway STM32G474" (at 286 72 0) (effects (font (size 1.4 1.4)) (justify left top)))
+(sheet (at 281 63) (size 112 27) (stroke (width 0) (type solid)) (fill (color 0 0 0 0)) (property "Sheetname" "Gateway STM32G473" (at 281 62 0) (effects (font (size 1.27 1.27)) (justify left bottom))) (property "Sheetfile" "gateway.kicad_sch" (at 281 91 0) (effects (font (size 1.0 1.0)) (justify left top))) (instances (project "board1" (path "/ab028fb1-c655-584d-9b32-a6ba9517f8a2" (page "4")))))
+(text "04  Gateway STM32G473" (at 286 72 0) (effects (font (size 1.4 1.4)) (justify left top)))
 (sheet (at 25 106) (size 112 27) (stroke (width 0) (type solid)) (fill (color 0 0 0 0)) (property "Sheetname" "SAM0" (at 25 105 0) (effects (font (size 1.27 1.27)) (justify left bottom))) (property "Sheetfile" "sam0.kicad_sch" (at 25 134 0) (effects (font (size 1.0 1.0)) (justify left top))) (instances (project "board1" (path "/ab028fb1-c655-584d-9b32-a6ba9517f8a2" (page "5")))))
 (text "05  SAM0" (at 30 115 0) (effects (font (size 1.4 1.4)) (justify left top)))
@@
 (text "11  Test access" (at 30 201 0) (effects (font (size 1.4 1.4)) (justify left top)))
 (text "CAN A/B: GW + SAM0 + SAM1 + SAM2, eight PHYs.\nUART_MD: four receivers; one LV125 channel per transmitter.\nSAM ring: SAM0 -> SAM1 -> SAM2 -> SAM0.\nEach MCU: SWD, private debug UART, SYNC/TRIG and EVENT0/1." (at 155 201 0) (effects (font (size 1.35 1.35)) (justify left top)))
-(text "Named global nets join sheets; local analog nets stay within their sheet.\nReview PDF and checks describe draft-capture evidence. ERC, layout/DRC\nand hardware bring-up are separate stages. No PCB layout yet." (at 25 256 0) (effects (font (size 1.2 1.2)) (justify left top)))
+(text "Named global nets join sheets; local analog nets stay within their sheet.\nReview PDF and checks describe draft-capture evidence. ERC, layout/DRC\nand hardware bring-up are separate stages. Initial PCB placement is unrouted." (at 25 256 0) (effects (font (size 1.2 1.2)) (justify left top)))
 (sheet_instances (path "/" (page "1")))
 )
