File: boards/board1/kicad/gateway.kicad_sch (KiCad schematic)
At the start: 27 parts, among them J2 GW timing/debug, J3 GW SWD, U7 STM32G474RBT6, Y2 12MHz / CL20p

Commit message: High-level layout done
Parts:
- C35, C36: MPN C0805C330F5GACTU -> CC0805FRNPO9BN330
- U7: value STM32G474RBT6 -> STM32G473RBT6; symbol MCU_ST_STM32G4:STM32G474RBTx -> MCU_ST_STM32G4:STM32G473RBTx; MPN STM32G474RBT6 -> STM32G473RBT6
Other:
- note added: "GW / STM32G473RBT6"
- note removed: "GW / STM32G474RBT6"
Changed lines of the file:
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@@
 (kicad_sch (version 20230121) (generator ws_hardware_capture) (paper "A3")
 (title_block (title "Board 1 - GW MCU, debug and timing") (date "2026-09-07") (rev "A-draft") (company "WireSpaces") (comment 1 "Rev A complete schematic draft - no PCB layout"))
-(text "GW / STM32G474RBT6" (at 20 20 0) (effects (font (size 2 2)) (justify left top)))
+(text "GW / STM32G473RBT6" (at 20 20 0) (effects (font (size 2 2)) (justify left top)))
 (text "TIMING / TEXT DEBUG" (at 218 20 0) (effects (font (size 1.7 1.7)) (justify left top)))
 (text "INDEPENDENT SWD" (at 318 126 0) (effects (font (size 1.6 1.6)) (justify left top)))
-(symbol (lib_id "MCU_ST_STM32G4:STM32G474RBTx") (at 100 107 0) (unit 1) (in_bom yes) (on_board yes) (dnp no)
+(symbol (lib_id "MCU_ST_STM32G4:STM32G473RBTx") (at 100 107 0) (unit 1) (in_bom yes) (on_board yes) (dnp no)
 (property "Reference" "U7" (at 78 45 0) (effects (font (size 1.15 1.15))))
-(property "Value" "STM32G474RBT6" (at 120 45 0) (effects (font (size 1.0 1.0))))
+(property "Value" "STM32G473RBT6" (at 120 45 0) (effects (font (size 1.0 1.0))))
 (property "Footprint" "Package_QFP:LQFP-64_10x10mm_P0.5mm" (at 100 107 0) (effects (font (size 1.0 1.0)) hide))
 (property "Datasheet" "https://www.st.com/resource/en/datasheet/stm32g474rb.pdf" (at 100 107 0) (effects (font (size 1.0 1.0)) hide))
 (property "BOM_ID" "B1-B001" (at 100 107 0) (effects (font (size 1.0 1.0)) hide))
-(property "MPN" "STM32G474RBT6" (at 100 107 0) (effects (font (size 1.0 1.0)) hide))
+(property "MPN" "STM32G473RBT6" (at 100 107 0) (effects (font (size 1.0 1.0)) hide))
 (property "Manufacturer" "STMicroelectronics" (at 100 107 0) (effects (font (size 1.0 1.0)) hide))
 (pin "1")
@@
 (property "Datasheet" "~" (at 212 246 0) (effects (font (size 1.0 1.0)) hide))
 (property "BOM_ID" "B1-B042" (at 212 246 0) (effects (font (size 1.0 1.0)) hide))
-(property "MPN" "C0805C330F5GACTU" (at 212 246 0) (effects (font (size 1.0 1.0)) hide))
+(property "MPN" "CC0805FRNPO9BN330" (at 212 246 0) (effects (font (size 1.0 1.0)) hide))
 (property "Manufacturer" "KEMET" (at 212 246 0) (effects (font (size 1.0 1.0)) hide))
 (pin "1")
@@
 (property "Datasheet" "~" (at 252 246 0) (effects (font (size 1.0 1.0)) hide))
 (property "BOM_ID" "B1-B042" (at 252 246 0) (effects (font (size 1.0 1.0)) hide))
-(property "MPN" "C0805C330F5GACTU" (at 252 246 0) (effects (font (size 1.0 1.0)) hide))
+(property "MPN" "CC0805FRNPO9BN330" (at 252 246 0) (effects (font (size 1.0 1.0)) hide))
 (property "Manufacturer" "KEMET" (at 252 246 0) (effects (font (size 1.0 1.0)) hide))
 (pin "1")
