File: boards/board1/kicad/sam1.kicad_sch (KiCad schematic)
At the start: 25 parts, among them J6 SAM1 timing/debug, J7 SAM1 SWD, U9 ATSAMC21G17A-AUT, Y4 12MHz / CL20p

Commit message: High-level layout done
Parts:
- C55, C56: MPN C0805C330F5GACTU -> CC0805FRNPO9BN330
Changed lines of the file:
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@@
 (property "Datasheet" "~" (at 212 246 0) (effects (font (size 1.0 1.0)) hide))
 (property "BOM_ID" "B1-B043" (at 212 246 0) (effects (font (size 1.0 1.0)) hide))
-(property "MPN" "C0805C330F5GACTU" (at 212 246 0) (effects (font (size 1.0 1.0)) hide))
+(property "MPN" "CC0805FRNPO9BN330" (at 212 246 0) (effects (font (size 1.0 1.0)) hide))
 (property "Manufacturer" "KEMET" (at 212 246 0) (effects (font (size 1.0 1.0)) hide))
 (pin "1")
@@
 (property "Datasheet" "~" (at 252 246 0) (effects (font (size 1.0 1.0)) hide))
 (property "BOM_ID" "B1-B043" (at 252 246 0) (effects (font (size 1.0 1.0)) hide))
-(property "MPN" "C0805C330F5GACTU" (at 252 246 0) (effects (font (size 1.0 1.0)) hide))
+(property "MPN" "CC0805FRNPO9BN330" (at 252 246 0) (effects (font (size 1.0 1.0)) hide))
 (property "Manufacturer" "KEMET" (at 252 246 0) (effects (font (size 1.0 1.0)) hide))
 (pin "1")
