File: boards/board1/kicad/sam2.kicad_sch (KiCad schematic)
At the start: 25 parts, among them J8 SAM2 timing/debug, J9 SAM2 SWD, U10 ATSAMC21G17A-AUT, Y5 12MHz / CL20p

Commit message: High-level layout done
Parts:
- C65, C66: MPN C0805C330F5GACTU -> CC0805FRNPO9BN330
Changed lines of the file:
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@@
 (property "Datasheet" "~" (at 212 246 0) (effects (font (size 1.0 1.0)) hide))
 (property "BOM_ID" "B1-B043" (at 212 246 0) (effects (font (size 1.0 1.0)) hide))
-(property "MPN" "C0805C330F5GACTU" (at 212 246 0) (effects (font (size 1.0 1.0)) hide))
+(property "MPN" "CC0805FRNPO9BN330" (at 212 246 0) (effects (font (size 1.0 1.0)) hide))
 (property "Manufacturer" "KEMET" (at 212 246 0) (effects (font (size 1.0 1.0)) hide))
 (pin "1")
@@
 (property "Datasheet" "~" (at 252 246 0) (effects (font (size 1.0 1.0)) hide))
 (property "BOM_ID" "B1-B043" (at 252 246 0) (effects (font (size 1.0 1.0)) hide))
-(property "MPN" "C0805C330F5GACTU" (at 252 246 0) (effects (font (size 1.0 1.0)) hide))
+(property "MPN" "CC0805FRNPO9BN330" (at 252 246 0) (effects (font (size 1.0 1.0)) hide))
 (property "Manufacturer" "KEMET" (at 252 246 0) (effects (font (size 1.0 1.0)) hide))
 (pin "1")
