File: boards/board1/kicad/usb_bridge.kicad_sch (KiCad schematic)
At the start: 30 parts, among them U4 FT232HL-REEL, U5 AT93C56B-SSHM-B, U6 SN74LV125APWR, Y1 12MHz / CL18p

Commit message: First draft finished
Other:
- note added: "GW_* directions are from the MCU. TX/RX idle high; CTS_N inactive high. All /OE pins directly use PWREN_N (ADR-040). These four GW nets connect to the gateway MCU sheet."
- note removed: "GW_* directions are from the MCU. TX/RX idle high; CTS_N inactive high. All /OE pins directly use PWREN_N (ADR-040). These four GW nets end at the next capture stage."

Commit message: High-level layout done
Parts:
- C12, C13: MPN C0805C270F5GACTU -> CC0805FRNPO9BN270
